Commit message: urdf fix. readme updated

File: raisim_gym/env/env/ANYmal/ANYmal_bear2/anymal.urdf (robot description, URDF)
Before this commit: robot anymal, 30 links, 29 joints
Links:
- link LF_FOOT: geometry collision sphere radius=0.038
- link LH_FOOT: geometry collision sphere radius=0.038
- link RF_FOOT: geometry collision sphere radius=0.038
- link RH_FOOT: geometry collision sphere radius=0.038
